Commit message: Robot navigates successfully. Navigation and keyboard control don't work together.

File: turtlebot3_gazebo/descriptions/gazebo_control.xacro (robot description, xacro)
@@ -2,7 +2,5 @@
 <robot xmlns:xacro="http://www.ros.org/wiki/xacro">
     <gazebo>
-        <plugin name="gazebo_ros2_diff_drive" filename="libgazebo_ros_diff_drive.so">
-            <namespace>/</namespace>
-            <remapping>cmd_vel:=/cmd_vel</remapping>
+        <plugin name="diff_drive" filename="libgazebo_ros_diff_drive.so">
             <!-- Wheel -->
             <left_joint>left_wheel_joint</left_joint>

File: turtlebot3_gazebo/descriptions/lidar.xacro (robot description, xacro)
@@ -2,10 +2,11 @@
 <robot xmlns:xacro="http://www.ros.org/wiki/xacro">
     <!-- REAR LIDAR-->
-    <joint name="laser_joint_r" type="fixed">
+    <!-- FRONT LIDAR-->
+    <joint name="laser_joint_f" type="fixed">
         <parent link="chassis" />
-        <child link="laser_frame_r" />
-        <origin xyz="0.1 0 0.23" rpy="0 0 ${pi}" />
+        <child link="laser_frame" />
+        <origin xyz="0.72 0 0.23" rpy="0 0 0" />
     </joint>
-    <link name="laser_frame_r">
+    <link name="laser_frame">
         <visual>
             <geometry>
@@ -23,55 +24,5 @@
         </xacro:inertial_cylinder>
     </link>
-    <gazebo reference="laser_frame_r">
-        <material>Gazebo/Red</material>
-        <sensor name="laser_r" type="ray">
-            <pose> 0 0 0 0 0 0 </pose>
-            <visualize>true</visualize>
-            <update_rate>10</update_rate>
-            <ray>
-                <scan>
-                    <horizontal>
-                        <samples>180</samples>
-                        <min_angle>-2.0</min_angle>
-                        <max_angle>2.0</max_angle>
-                    </horizontal>
-                </scan>
-                <range>
-                    <min>0.4</min>
-                    <max>12</max>
-                </range>
-            </ray>
-            <plugin name="laser_controller_r" filename="libgazebo_ros_ray_sensor.so">
-                <ros>
-                    <argument>--ros-args --remap ~/out:=scan_r</argument>
-                </ros>
-                <output_type>sensor_msgs/LaserScan</output_type>
-                <frame_name>laser_frame_r</frame_name>
-            </plugin>
-        </sensor>
-    </gazebo>
-    <!-- FRONT LIDAR-->
-    <joint name="laser_joint_f" type="fixed">
-        <parent link="chassis" />
-        <child link="laser_frame_f" />
-        <origin xyz="0.72 0 0.23" rpy="0 0 0" />
-    </joint>
-    <link name="laser_frame_f">
-        <visual>
-            <geometry>
-                <cylinder radius="0.05" length="0.04" />
-            </geometry>
-            <material name="red" />
-        </visual>
-        <collision>
-            <geometry>
-                <cylinder radius="0.05" length="0.04" />
-            </geometry>
-        </collision>
-        <xacro:inertial_cylinder mass="0.1" length="0.04" radius="0.05">
-            <origin xyz="0 0 0" rpy="0 0 0" />
-        </xacro:inertial_cylinder>
-    </link>
-    <gazebo reference="laser_frame_f">
+    <gazebo reference="laser_frame">
         <material>Gazebo/Red</material>
         <sensor name="laser_f" type="ray">
@@ -83,6 +34,6 @@
                     <horizontal>
                         <samples>180</samples>
-                        <min_angle>-2.0</min_angle>
-                        <max_angle>2.0</max_angle>
+                        <min_angle>-2</min_angle>
+                        <max_angle>2</max_angle>
                     </horizontal>
                 </scan>
@@ -94,8 +45,8 @@
             <plugin name="laser_controller_f" filename="libgazebo_ros_ray_sensor.so">
                 <ros>
-                    <argument>--ros-args --remap ~/out:=scan_f</argument>
+                    <argument>~/out:=scan</argument>
                 </ros>
                 <output_type>sensor_msgs/LaserScan</output_type>
-                <frame_name>laser_frame_f</frame_name>
+                <frame_name>laser_frame</frame_name>
             </plugin>
         </sensor>

File: turtlebot3_gazebo/descriptions/robot_core.xacro (robot description, xacro)
@@ -26,5 +26,5 @@
                 <box size="0.82 0.65 0.23" />
             </geometry>
-            <material name="white" />
+            <material name="orange" />
         </visual>
         <collision>
@@ -39,5 +39,5 @@
     </link>
     <gazebo reference="chassis">
-        <material>Gazebo/White</material>
+        <material>Gazebo/Orange</material>
     </gazebo>
     <!-- LEFT WHEEL LINK -->

File: turtlebot3_gazebo/descriptions/ros2_control.xacro (robot description, xacro)
@@ -28,4 +28,5 @@
         <plugin name="gazebo_ros2_control" filename="libgazebo_ros2_control.so">
             <parameters>$(find turtlebot3_gazebo)/config/my_controllers.yaml</parameters>
+            <parameters>$(find turtlebot3_gazebo)/config/gaz_ros2_ctl_use_sim.yaml</parameters>
         </plugin>
     </gazebo>
