Commit message: use_sim_time is set to false and launch file for real robot added

File: turtlebot3_gazebo/descriptions/ros2_control.xacro (robot description, xacro)
@@ -2,5 +2,29 @@
 <robot xmlns:xacro="http://www.ros.org/wiki/xacro">
     <!-- Hardware Interface for the Controller Manager-->
-    <ros2_control name="GazeboSystem" type="system">
+    <ros2_control name="RealRobot" type="system">
+        <hardware>
+            <plugin>canopen_driver/CanOpenDriver</plugin>
+            <param name="left_wheel_name">left_wheel_joint</param>
+            <param name="right_wheel_name">right_wheel_joint</param>
+            <param name="device">/dev/ttyACM0</param>
+        </hardware>
+        <joint name="left_wheel_joint">
+            <command_interface name="velocity">
+                <param name="min">-15</param>
+                <param name="max">15</param>
+            </command_interface>
+            <state_interface name="velocity" />
+            <state_interface name="position" />
+        </joint>
+        <joint name="right_wheel_joint">
+            <command_interface name="velocity">
+                <param name="min">-15</param>
+                <param name="max">15</param>
+            </command_interface>
+            <state_interface name="velocity" />
+            <state_interface name="position" />
+        </joint>
+    </ros2_control>
+    <!-- <ros2_control name="GazeboSystem" type="system">
         <hardware>
             <plugin>gazebo_ros2_control/GazeboSystem</plugin>
@@ -22,5 +46,5 @@
             <state_interface name="position" />
         </joint>
-    </ros2_control>
+    </ros2_control> -->
     <!-- gazebo_ros2_control is a Gazebo pluging that integrats ros2_control with Gazebo,
     (tells Gazebo to use ros2_control)-->
