Commit message: Algorithm for attach to docking station corrected. Wheel radius and gear ratio coefficients added.

File: turtlebot3_gazebo/descriptions/robot_core.xacro (robot description, xacro)
@@ -45,5 +45,5 @@
         <parent link="base_link" />
         <child link="left_wheel" />
-        <origin xyz="0 0.303 -0.075" rpy="-${pi/2} 0 0" />
+        <origin xyz="0 0.295 -0.075" rpy="-${pi/2} 0 0" />
         <axis xyz="0 0 1" />
     </joint>
@@ -51,5 +51,5 @@
         <visual>
             <geometry>
-                <cylinder radius="0.075" length="0.045" />
+                <cylinder radius="0.074" length="0.045" />
             </geometry>
             <material name="blue" />
@@ -57,8 +57,8 @@
         <collision>
             <geometry>
-                <sphere radius="0.075" />
-            </geometry>
-        </collision>
-        <xacro:inertial_cylinder mass="0.1" length="0.045" radius="0.075">
+                <sphere radius="0.074" />
+            </geometry>
+        </collision>
+        <xacro:inertial_cylinder mass="0.1" length="0.045" radius="0.074">
             <origin xyz="0 0 0" rpy="0 0 0" />
         </xacro:inertial_cylinder>
@@ -71,5 +71,5 @@
         <parent link="base_link" />
         <child link="right_wheel" />
-        <origin xyz="0 -0.303 -0.075" rpy="${pi/2} 0 0" />
+        <origin xyz="0 -0.295 -0.075" rpy="${pi/2} 0 0" />
         <axis xyz="0 0 -1" />
     </joint>
@@ -77,5 +77,5 @@
         <visual>
             <geometry>
-                <cylinder radius="0.075" length="0.045" />
+                <cylinder radius="0.074" length="0.045" />
             </geometry>
             <material name="blue" />
@@ -83,8 +83,8 @@
         <collision>
             <geometry>
-                <sphere radius="0.075" />
-            </geometry>
-        </collision>
-        <xacro:inertial_cylinder mass="0.1" length="0.045" radius="0.075">
+                <sphere radius="0.074" />
+            </geometry>
+        </collision>
+        <xacro:inertial_cylinder mass="0.1" length="0.045" radius="0.074">
             <origin xyz="0 0 0" rpy="0 0 0" />
         </xacro:inertial_cylinder>
