Commit message: some updates to xacro

File: caspi_bot/descriptions/lidar.xacro (robot description, xacro)
@@ -6,5 +6,5 @@
         <parent link="chassis" />
         <child link="laser_frame" />
-        <origin xyz="0.72 0 0.23" rpy="0 0 0" />
+        <origin xyz="0.82 0 0.23" rpy="0 0 0" />
     </joint>
     <link name="laser_frame">
@@ -39,6 +39,6 @@
                 </scan>
                 <range>
-                    <min>0.4</min>
-                    <max>12</max>
+                    <min>0.06</min>
+                    <max>4</max>
                 </range>
             </ray>

File: caspi_bot/descriptions/robot_core.xacro (robot description, xacro)
@@ -34,5 +34,5 @@
             </geometry>
         </collision>
-        <xacro:inertial_box mass="0.5" x="0.3" y="0.3" z="0.15">
+        <xacro:inertial_box mass="15.0" x="0.3" y="0.3" z="0.15">
             <origin xyz="0.15 0 0.075" rpy="0 0 0" />
         </xacro:inertial_box>
@@ -60,5 +60,5 @@
             </geometry>
         </collision>
-        <xacro:inertial_cylinder mass="0.1" length="0.045" radius="0.074">
+        <xacro:inertial_cylinder mass="2.0" length="0.045" radius="0.074">
             <origin xyz="0 0 0" rpy="0 0 0" />
         </xacro:inertial_cylinder>
@@ -86,5 +86,5 @@
             </geometry>
         </collision>
-        <xacro:inertial_cylinder mass="0.1" length="0.045" radius="0.074">
+        <xacro:inertial_cylinder mass="2.0" length="0.045" radius="0.074">
             <origin xyz="0 0 0" rpy="0 0 0" />
         </xacro:inertial_cylinder>
@@ -111,5 +111,5 @@
             </geometry>
         </collision>
-        <xacro:inertial_cylinder mass="0.1" length="0.045" radius="0.075">
+        <xacro:inertial_cylinder mass="1.0" length="0.045" radius="0.075">
             <origin xyz="0 0 0" rpy="0 0 0" />
         </xacro:inertial_cylinder>
@@ -138,5 +138,5 @@
             </geometry>
         </collision>
-        <xacro:inertial_cylinder mass="0.1" length="0.045" radius="0.075">
+        <xacro:inertial_cylinder mass="1.0" length="0.045" radius="0.075">
             <origin xyz="0 0 0" rpy="0 0 0" />
         </xacro:inertial_cylinder>
@@ -165,5 +165,5 @@
             </geometry>
         </collision>
-        <xacro:inertial_cylinder mass="0.1" length="0.045" radius="0.075">
+        <xacro:inertial_cylinder mass="1.0" length="0.045" radius="0.075">
             <origin xyz="0 0 0" rpy="0 0 0" />
         </xacro:inertial_cylinder>
@@ -192,5 +192,5 @@
             </geometry>
         </collision>
-        <xacro:inertial_cylinder mass="0.1" length="0.045" radius="0.075">
+        <xacro:inertial_cylinder mass="1.0" length="0.045" radius="0.075">
             <origin xyz="0 0 0" rpy="0 0 0" />
         </xacro:inertial_cylinder>
